Commit message: 机械臂控制系统修改

File: ACETeleop-main/ace_teleop/assets/gen_72_b_description/urdf/GEN72_franka.urdf (robot description, URDF)
Before this commit: robot GEN72, 29 links, 28 joints
Links:
- link l_Link1: geometry collision mesh filename=../meshes/Link1.STL; visual mesh filename=../meshes/Link1.STL
- link l_Link2: geometry collision mesh filename=../meshes/Link2.STL; visual mesh filename=../meshes/Link2.STL
- link l_Link3: geometry collision mesh filename=../meshes/Link3.STL; visual mesh filename=../meshes/Link3.STL
- link l_Link4: geometry collision mesh filename=../meshes/Link4.STL; visual mesh filename=../meshes/Link4.STL
- link l_Link5: geometry collision mesh filename=../meshes/Link5.STL; visual mesh filename=../meshes/Link5.STL
- link l_Link6: geometry collision mesh filename=../meshes/Link6.STL; visual mesh filename=../meshes/Link6.STL
- link l_Link7: geometry collision mesh filename=../meshes/Link7.STL; visual mesh filename=../meshes/Link7.STL
- link l_base_link: geometry collision mesh filename=../meshes/base_link.STL; visual mesh filename=../meshes/base_link.STL
- link l_panda_hand: geometry collision mesh filename=/home/s402/ACE/ACETeleop-main/ace_teleop/assets/franka/fran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; visual mesh filename=../../franka/franka_description/meshes/visual/hand.glb
- link r_Link1: geometry collision mesh filename=../meshes/Link1.STL; visual mesh filename=../meshes/Link1.STL
- link r_Link2: geometry collision mesh filename=../meshes/Link2.STL; visual mesh filename=../meshes/Link2.STL
- link r_Link3: geometry collision mesh filename=../meshes/Link3.STL; visual mesh filename=../meshes/Link3.STL
- link r_Link4: geometry collision mesh filename=../meshes/Link4.STL; visual mesh filename=../meshes/Link4.STL
- link r_Link5: geometry collision mesh filename=../meshes/Link5.STL; visual mesh filename=../meshes/Link5.STL
- link r_Link6: geometry collision mesh filename=../meshes/Link6.STL; visual mesh filename=../meshes/Link6.STL
- link r_Link7: geometry collision mesh filename=../meshes/Link7.STL; visual mesh filename=../meshes/Link7.STL
- link r_base_link: geometry collision mesh filename=../meshes/base_link.STL; visual mesh filename=../meshes/base_link.STL
